Commit message: configurations, tracking, central system, pid, etc.

File: pesat_resources/urdf/bebop2_fixed_camera.urdf (robot description, URDF)
Before this commit: robot bebop2, 14 links, 13 joints
Links:
- removed link bebop2/camera_rotator_base_link
Joints:
- removed joint bebop2/camera_rotator_base_joint
- joint bebop2/camera_base_joint: axis 0 0 1 -> (none); limit lower=-0.523598775598 upper=0.523598775598 effort=0.02 velocity=0.02 -> (none); parent bebop2/camera_rotator_base_link -> bebop2/base_link; type revolute -> fixed
