Commit message: big update

File: pesat_resources/urdf/ball.urdf (robot description, URDF)
Before this commit: robot simple_ball, 1 links, 0 joints
Links:
- removed link ball
- added link target/base_link, mass 1.0; collision sphere radius=1; visual sphere radius=1

File: pesat_resources/urdf/bebop2.urdf (robot description, URDF)
Before this commit: robot bebop2, 14 links, 13 joints
Links:
- added link bebop2/sonar_sensor_base_link, mass 1e-05; collision box size=0.001 0.001 0.001; visual box size=0.001 0.001 0.001
Joints:
- added joint bebop2/sonar_sensor_base_joint: type revolute, parent bebop2/base_link, child bebop2/sonar_sensor_base_link, origin xyz=0.1 0 0 rpy=0 1.5707963268 0, limit lower=0 upper=0 effort=0 velocity=0
- joint bebop2/camera_base_joint: origin xyz=0.1 0 0 rpy=0 0 0 -> xyz=0 0 0 rpy=0 0 0

File: pesat_resources/urdf/bebop2.xacro (robot description, xacro)
@@ -145,3 +145,22 @@
       <origin xyz="0.1 0 0" rpy="0 0 0" />
   </xacro:rotable_camera_macro>
+  <xacro:sonar_sensor_plugin_macro
+      namespace="${namespace}"
+      parent_link="${namespace}/base_link"
+      sonar_sensor_suffix="base"
+      update_rate="50.0"
+      min_distance="0.06"
+      max_distance="50.0"
+      noise_mean="0.005"
+      enable_visual="true"
+      sonar_topic="sensors/sonar"
+      mass_sonar_sensor="1e-5"
+      range_resolution="0.02"
+      scan_resolution="1.0"
+      samples="10"
+      angle="0.14835"
+      fov="0.2967">
+      <box size="0.001 0.001 0.001" />
+      <origin xyz="0.1 0 0" rpy="0 ${pi/2} 0" />
+  </xacro:sonar_sensor_plugin_macro>
 </robot>

File: pesat_resources/urdf/component_snippets.xacro (robot description, xacro)
@@ -32,4 +32,82 @@
     </gazebo>
   </xacro:macro>
+  <!-- Macro to add sonar sensor. -->
+  <xacro:macro name="sonar_sensor_plugin_macro"
+    params="namespace sonar_sensor_suffix parent_link sonar_topic
+      mass_sonar_sensor angle fov noise_mean min_distance max_distance enable_visual
+      samples update_rate scan_resolution range_resolution *geometry *origin">
+    <!-- Sonar sensor link -->
+    <link name="${namespace}/sonar_sensor_${sonar_sensor_suffix}_link">
+      <collision>
+        <origin xyz="0 0 0" rpy="0 0 0" />
+        <geometry>
+          <xacro:insert_block name="geometry" />
+        </geometry>
+      </collision>
+      <xacro:if value="${enable_visual}">
+        <visual>
+          <origin xyz="0 0 0" rpy="0 0 0" />
+          <geometry>
+            <xacro:insert_block name="geometry" />
+          </geometry>
+          <material name="red" />
+        </visual>
+      </xacro:if>
+      <inertial>
+        <mass value="${mass_sonar_sensor}" />
+        <origin xyz="0 0 0" rpy="0 0 0" />
+        <inertia ixx="1e-6" ixy="0" ixz="0" iyy="1e-6" iyz="0" izz="1e-6" />
+      </inertial>
+    </link>
+    <!-- Sonar sensor joint -->
+    <joint name="${namespace}/sonar_sensor_${sonar_sensor_suffix}_joint" type="revolute">
+      <xacro:insert_block name="origin" />
+      <parent link="${parent_link}" />
+      <child link="${namespace}/sonar_sensor_${sonar_sensor_suffix}_link" />
+      <limit upper="0" lower="0" effort="0" velocity="0" />
+    </joint>
+    <!-- Sonar sensor gazebo -->
+    <gazebo reference="${namespace}/sonar_sensor_${sonar_sensor_suffix}_link">
+	   <sensor type="ray" name="sonar">
+	      <pose>0 0 0 0 0 0</pose>
+	      <visualize>${enable_visual}</visualize>
+	      <update_rate>${update_rate}</update_rate>
+	      <ray>
+		 <scan>
+		    <horizontal>
+		       <!-- default angle 10 -->
+		       <samples>${samples}</samples>
+		       <!-- default angle 1 -->
+		       <resolution>${scan_resolution}</resolution>
+		       <!-- default angle 0.14835 -->
+		       <min_angle>-${angle}</min_angle>
+		       <max_angle>${angle}</max_angle>
+		    </horizontal>
+		    <vertical>
+		       <samples>${samples}</samples>
+		       <resolution>${scan_resolution}</resolution>
+		       <min_angle>-${angle}</min_angle>
+		       <max_angle>${angle}</max_angle>
+		    </vertical>
+		 </scan>
+		 <range>
+		    <min>${min_distance}</min>
+		    <max>${max_distance}</max>
+		    <resolution>${range_resolution}</resolution>
+		 </range>
+	      </ray>
+	      <plugin filename="libgazebo_ros_range.so" name="gazebo_ros_range">
+	       <!-- default 0.005 -->
+		 <gaussianNoise>${noise_mean}</gaussianNoise>
+		 <alwaysOn>true</alwaysOn>
+		 <updateRate>${update_rate}</updateRate>
+		 <topicName>${sonar_topic}</topicName>
+		 <frameName>${namespace}/sonar_sensor_${sonar_sensor_suffix}_link</frameName>
+		 <radiation>ultrasound</radiation>
+		 <fov>${fov}</fov> <!-- 0.2967 -->
+	      </plugin>
+	   </sensor>
+   </gazebo>
+  </xacro:macro>
   <!--  Macro to add a rotable camera  -->
   <!-- base_link - revolute joint -> camera_rotator_base_link - revolute joint -> camera_base_link - fixed joint -> camera_optical_base_link  -->
@@ -90,5 +168,5 @@
     </joint>
     <joint name="${namespace}/camera_${camera_suffix}_joint" type="revolute">
-      <xacro:insert_block name="origin" />
+      <origin xyz="0 0 0" rpy="0 0 0" />
       <parent link="${namespace}/camera_rotator_${camera_suffix}_link" />
       <child link="${namespace}/camera_${camera_suffix}_link" />
@@ -146,9 +224,9 @@
       <type>transmission_interface/SimpleTransmission</type>
       <actuator name="motor_vertical">
-        <hardwareInterface>hardware_interface/VelocityJointInterface</hardwareInterface>
+        <hardwareInterface>hardware_interface/PositionJointInterface</hardwareInterface>
         <mechanicalReduction>1</mechanicalReduction>
       </actuator>
       <joint name="${namespace}/camera_rotator_${camera_suffix}_joint">
-        <hardwareInterface>hardware_interface/VelocityJointInterface</hardwareInterface>
+        <hardwareInterface>hardware_interface/PositionJointInterface</hardwareInterface>
       </joint>
     </transmission>
@@ -156,9 +234,9 @@
       <type>transmission_interface/SimpleTransmission</type>
       <actuator name="motor_horizontal">
-        <hardwareInterface>hardware_interface/VelocityJointInterface</hardwareInterface>
+        <hardwareInterface>hardware_interface/PositionJointInterface</hardwareInterface>
         <mechanicalReduction>1</mechanicalReduction>
       </actuator>
       <joint name="${namespace}/camera_${camera_suffix}_joint">
-        <hardwareInterface>hardware_interface/VelocityJointInterface</hardwareInterface>
+        <hardwareInterface>hardware_interface/PositionJointInterface</hardwareInterface>
       </joint>
     </transmission>
