Commit message: Update

File: pesat_resources/urdf/bebop2.urdf (robot description, URDF)
Before this commit: robot bebop2, 15 links, 14 joints
Joints:
- joint bebop2/camera_base_joint: axis 0 0 1 -> 0 1 0; limit lower=-0.523598775598 upper=0.523598775598 effort=0.02 velocity=0.02 -> lower=-0.523598775598 upper=0.523598775598 effort=0.02 velocity=1.0
- joint bebop2/camera_rotator_base_joint: axis 0 1 0 -> 0 0 1; limit lower=-0.523598775598 upper=0.523598775598 effort=0.02 velocity=0.02 -> lower=-0.523598775598 upper=0.523598775598 effort=0.02 velocity=1.0

File: pesat_resources/urdf/component_snippets.xacro (robot description, xacro)
@@ -164,5 +164,5 @@
       <parent link="${parent_link}" />
       <child link="${namespace}/camera_rotator_${camera_suffix}_link" />
-      <axis xyz="0 1 0"/>
+      <axis xyz="0 0 1"/>
       <limit lower="-${pi/6}" upper="${pi/6}" effort="2.0" velocity="2.00" />
     </joint>
@@ -171,5 +171,5 @@
       <parent link="${namespace}/camera_rotator_${camera_suffix}_link" />
       <child link="${namespace}/camera_${camera_suffix}_link" />
-      <axis xyz="0 0 1"/>
+      <axis xyz="0 1 0"/>
       <limit lower="-${pi/6}" upper="${pi/6}" effort="2.0" velocity="2.0" />
     </joint>
